File: EtherDue.sch (KiCad schematic (older format))
At the start: 29 parts, among them P101 CONN_02X04, P102 MSTBV3, P103 MSTBV3, P104 MSTBV6, Q101 IPB020NE7N3G, Q102 IPB020NE7N3G, U101 AD7415, U1701 MCP6H04

Commit message: Rev B. Layout - Gerber/BOM need to be reexported
Parts:
- R101, R102: value Shunt -> Shunt 10mOhm
Changed lines of the file:
@@
 LIBS:w_transistor
 LIBS:w_logic
+LIBS:w_memory
 EELAYER 25 0
 EELAYER END
@@
 $EndComp
 $Comp
-L GND-RESCUE-EtherDue #PWR118
+L GND-RESCUE-EtherDue #PWR01
 U 1 1 54FF834A
 P 15550 3200
-F 0 "#PWR118" H 15550 2950 60  0001 C CNN
+F 0 "#PWR01" H 15550 2950 60  0001 C CNN
 F 1 "GND" H 15550 3050 60  0000 C CNN
 F 2 "" H 15550 3200 60  0000 C CNN
@@
 $EndComp
 $Comp
-L GND-RESCUE-EtherDue #PWR119
+L GND-RESCUE-EtherDue #PWR02
 U 1 1 55086BA7
 P 15550 4750
-F 0 "#PWR119" H 15550 4500 60  0001 C CNN
+F 0 "#PWR02" H 15550 4500 60  0001 C CNN
 F 1 "GND" H 15550 4600 60  0000 C CNN
 F 2 "" H 15550 4750 60  0000 C CNN
@@
 $EndComp
 $Comp
-L GND-RESCUE-EtherDue #PWR116
+L GND-RESCUE-EtherDue #PWR03
 U 1 1 550892B1
 P 15400 6800
-F 0 "#PWR116" H 15400 6550 60  0001 C CNN
+F 0 "#PWR03" H 15400 6550 60  0001 C CNN
 F 1 "GND" H 15400 6650 60  0000 C CNN
 F 2 "" H 15400 6800 60  0000 C CNN
@@
 $EndComp
 $Comp
-L GND-RESCUE-EtherDue #PWR115
+L GND-RESCUE-EtherDue #PWR04
 U 1 1 55097879
 P 15100 8200
-F 0 "#PWR115" H 15100 7950 60  0001 C CNN
+F 0 "#PWR04" H 15100 7950 60  0001 C CNN
 F 1 "GND" H 15100 8050 60  0000 C CNN
 F 2 "" H 15100 8200 60  0000 C CNN
@@
 SCL0-3
 $Comp
-L +3.3V #PWR101
+L +3.3V #PWR05
 U 1 1 54F2966F
 P 700 6800
-F 0 "#PWR101" H 700 6760 30  0001 C CNN
+F 0 "#PWR05" H 700 6760 30  0001 C CNN
 F 1 "+3.3V" H 700 6910 50  0000 C CNN
 F 2 "" H 700 6800 60  0000 C CNN
@@
 $EndComp
 $Comp
-L +5V #PWR102
+L +5V #PWR06
 U 1 1 54F2B047
 P 900 6950
-F 0 "#PWR102" H 900 6800 60  0001 C CNN
+F 0 "#PWR06" H 900 6800 60  0001 C CNN
 F 1 "+5V" H 900 7090 60  0000 C CNN
 F 2 "" H 900 6950 60  0000 C CNN
@@
 $EndComp
 $Comp
-L GND-RESCUE-EtherDue #PWR117
+L GND-RESCUE-EtherDue #PWR07
 U 1 1 54FB2A3C
 P 15500 8200
-F 0 "#PWR117" H 15500 7950 60  0001 C CNN
+F 0 "#PWR07" H 15500 7950 60  0001 C CNN
 F 1 "GND" H 15500 8050 60  0000 C CNN
 F 2 "" H 15500 8200 60  0000 C CNN
@@
 $EndComp
 $Comp
-L GND-RESCUE-EtherDue #PWR109
+L GND-RESCUE-EtherDue #PWR08
 U 1 1 55027291
 P 9700 2000
-F 0 "#PWR109" H 9700 1750 60  0001 C CNN
+F 0 "#PWR08" H 9700 1750 60  0001 C CNN
 F 1 "GND" H 9700 1850 60  0000 C CNN
 F 2 "" H 9700 2000 60  0000 C CNN
@@
 $EndComp
 $Comp
-L GND-RESCUE-EtherDue #PWR111
+L GND-RESCUE-EtherDue #PWR09
 U 1 1 550272B2
 P 10500 2250
-F 0 "#PWR111" H 10500 2000 60  0001 C CNN
+F 0 "#PWR09" H 10500 2000 60  0001 C CNN
 F 1 "GND" H 10500 2100 60  0000 C CNN
 F 2 "" H 10500 2250 60  0000 C CNN
@@
 P 14550 3300
 F 0 "R101" V 14630 3300 50  0000 C CNN
-F 1 "Shunt" V 14557 3301 50  0000 C CNN
+F 1 "Shunt 10mOhm" V 14557 3301 50  0000 C CNN
 F 2 "eagle-shunt:WSL4026" V 14480 3300 30  0001 C CNN
 F 3 "" H 14550 3300 30  0000 C CNN
@@
 P 14550 4850
 F 0 "R102" V 14630 4850 50  0000 C CNN
-F 1 "Shunt" V 14557 4851 50  0000 C CNN
+F 1 "Shunt 10mOhm" V 14557 4851 50  0000 C CNN
 F 2 "eagle-shunt:WSL4026" V 14480 4850 30  0001 C CNN
 F 3 "" H 14550 4850 30  0000 C CNN
@@
 $EndComp
 $Comp
-L GND-RESCUE-EtherDue #PWR112
+L GND-RESCUE-EtherDue #PWR010
 U 1 1 54FA8AB8
 P 12200 2300
-F 0 "#PWR112" H 12200 2050 60  0001 C CNN
+F 0 "#PWR010" H 12200 2050 60  0001 C CNN
 F 1 "GND" H 12200 2150 60  0000 C CNN
 F 2 "" H 12200 2300 60  0000 C CNN
@@
 	14150 2000 14150 2500
 $Comp
-L GND-RESCUE-EtherDue #PWR113
+L GND-RESCUE-EtherDue #PWR011
 U 1 1 550B8F13
 P 13150 1900
-F 0 "#PWR113" H 13150 1650 60  0001 C CNN
+F 0 "#PWR011" H 13150 1650 60  0001 C CNN
 F 1 "GND" H 13150 1750 60  0000 C CNN
 F 2 "" H 13150 1900 60  0000 C CNN
@@
 $EndComp
 $Comp
-L GND-RESCUE-EtherDue #PWR103
+L GND-RESCUE-EtherDue #PWR012
 U 1 1 5506D3DF
 P 7200 8350
-F 0 "#PWR103" H 7200 8100 60  0001 C CNN
+F 0 "#PWR012" H 7200 8100 60  0001 C CNN
 F 1 "GND" H 7200 8200 60  0000 C CNN
 F 2 "" H 7200 8350 60  0000 C CNN
@@
 $EndComp
 $Comp
-L GND-RESCUE-EtherDue #PWR104
+L GND-RESCUE-EtherDue #PWR013
 U 1 1 5506D3ED
 P 7600 8350
-F 0 "#PWR104" H 7600 8100 60  0001 C CNN
+F 0 "#PWR013" H 7600 8100 60  0001 C CNN
 F 1 "GND" H 7600 8200 60  0000 C CNN
 F 2 "" H 7600 8350 60  0000 C CNN
@@
 $EndComp
 $Comp
-L GND-RESCUE-EtherDue #PWR105
+L GND-RESCUE-EtherDue #PWR014
 U 1 1 55078E7F
 P 8150 9050
-F 0 "#PWR105" H 8150 8800 60  0001 C CNN
+F 0 "#PWR014" H 8150 8800 60  0001 C CNN
 F 1 "GND" H 8150 8900 60  0000 C CNN
 F 2 "" H 8150 9050 60  0000 C CNN
@@
 $EndComp
 $Comp
-L GND-RESCUE-EtherDue #PWR106
+L GND-RESCUE-EtherDue #PWR015
 U 1 1 55078E8D
 P 8550 9050
-F 0 "#PWR106" H 8550 8800 60  0001 C CNN
+F 0 "#PWR015" H 8550 8800 60  0001 C CNN
 F 1 "GND" H 8550 8900 60  0000 C CNN
 F 2 "" H 8550 9050 60  0000 C CNN
@@
 $EndComp
 $Comp
-L GND-RESCUE-EtherDue #PWR110
+L GND-RESCUE-EtherDue #PWR016
 U 1 1 55137138
 P 10250 3000
-F 0 "#PWR110" H 10250 2750 60  0001 C CNN
+F 0 "#PWR016" H 10250 2750 60  0001 C CNN
 F 1 "GND" H 10250 2850 60  0000 C CNN
 F 2 "" H 10250 3000 60  0000 C CNN
@@
 $EndComp
 $Comp
-L GND-RESCUE-EtherDue #PWR114
+L GND-RESCUE-EtherDue #PWR017
 U 1 1 55150219
 P 14450 2450
-F 0 "#PWR114" H 14450 2200 60  0001 C CNN
+F 0 "#PWR017" H 14450 2200 60  0001 C CNN
 F 1 "GND" H 14450 2300 60  0000 C CNN
 F 2 "" H 14450 2450 60  0000 C CNN
@@
 $EndComp
 $Comp
-L GND-RESCUE-EtherDue #PWR107
+L GND-RESCUE-EtherDue #PWR018
 U 1 1 5554E6ED
 P 8950 8400
-F 0 "#PWR107" H 8950 8150 60  0001 C CNN
+F 0 "#PWR018" H 8950 8150 60  0001 C CNN
 F 1 "GND" H 8950 8250 60  0000 C CNN
 F 2 "" H 8950 8400 60  0000 C CNN
@@
 $EndComp
 $Comp
-L GND-RESCUE-EtherDue #PWR108
+L GND-RESCUE-EtherDue #PWR019
 U 1 1 5554EF60
 P 8950 9100
-F 0 "#PWR108" H 8950 8850 60  0001 C CNN
+F 0 "#PWR019" H 8950 8850 60  0001 C CNN
 F 1 "GND" H 8950 8950 60  0000 C CNN
 F 2 "" H 8950 9100 60  0000 C CNN
