File: EtherDue_Ethernet.sch (KiCad schematic (older format))
At the start: 33 parts, among them IC601 W5100, Q601 2N7002, U602 HY931147C, U603 APX811-31UG-7, X601 TXC 7A 25MHz 18pF

Commit message: Rev B. Layout - Gerber/BOM need to be reexported
Parts:
- C604, C606, C608: value 10uF 6.3V A TANT -> 10u/25V/X7R
- L601, L602: value 1uH 250mA -> WE-CBF-742792093
Changed lines of the file:
@@
 LIBS:w_transistor
 LIBS:w_logic
+LIBS:w_memory
 EELAYER 25 0
 EELAYER END
@@
 $EndDescr
 $Comp
-L PWR_FLAG #FLG502
+L PWR_FLAG #FLG068
 U 1 1 51663F3F
 P 5950 6600
-F 0 "#FLG502" H 5950 6695 30  0001 C CNN
+F 0 "#FLG068" H 5950 6695 30  0001 C CNN
 F 1 "PWR_FLAG" H 5950 6780 30  0000 C CNN
 F 2 "" H 5950 6600 60  0001 C CNN
@@
 $EndComp
 $Comp
-L PWR_FLAG #FLG501
+L PWR_FLAG #FLG069
 U 1 1 51663F3A
 P 3950 6600
-F 0 "#FLG501" H 3950 6695 30  0001 C CNN
+F 0 "#FLG069" H 3950 6695 30  0001 C CNN
 F 1 "PWR_FLAG" H 3950 6780 30  0000 C CNN
 F 2 "" H 3950 6600 60  0001 C CNN
@@
 $EndComp
 $Comp
-L GND-RESCUE-EtherDue #PWR527
+L GND-RESCUE-EtherDue #PWR070
 U 1 1 51663F24
 P 10200 2350
-F 0 "#PWR527" H 10200 2350 30  0001 C CNN
+F 0 "#PWR070" H 10200 2350 30  0001 C CNN
 F 1 "GND" H 10200 2280 30  0001 C CNN
 F 2 "" H 10200 2350 60  0001 C CNN
@@
 /MASTER-RESET
 $Comp
-L +3.3V #PWR526
+L +3.3V #PWR071
 U 1 1 51663BD9
 P 9850 1100
-F 0 "#PWR526" H 9850 1060 30  0001 C CNN
+F 0 "#PWR071" H 9850 1060 30  0001 C CNN
 F 1 "+3.3V" H 9850 1210 30  0000 C CNN
 F 2 "" H 9850 1100 60  0001 C CNN
@@
 W5100 Reset on Poweron
 $Comp
-L +3.3V #PWR514
+L +3.3V #PWR072
 U 1 1 51663ACF
 P 4700 6600
-F 0 "#PWR514" H 4700 6560 30  0001 C CNN
+F 0 "#PWR072" H 4700 6560 30  0001 C CNN
 F 1 "+3.3V" H 4700 6710 30  0000 C CNN
 F 2 "" H 4700 6600 60  0001 C CNN
@@
 P 6100 7000
 F 0 "C608" H 6150 7100 50  0000 L CNN
-F 1 "10uF 6.3V A TANT" V 5950 6650 50  0000 L CNN
+F 1 "10u/25V/X7R" V 5950 6650 50  0000 L CNN
 F 2 "SMD_Packages:SMD-1206_Pol" H 6100 7000 60  0001 C CNN
 F 3 "" H 6100 7000 60  0001 C CNN
@@
 P 5500 6600
 F 0 "L602" H 5450 6700 40  0000 C CNN
-F 1 "1uH 250mA" H 5500 6550 40  0000 C CNN
+F 1 "WE-CBF-742792093" H 5500 6550 40  0000 C CNN
 F 2 "FT:0805" H 5500 6600 60  0001 C CNN
 F 3 "" H 5500 6600 60  0001 C CNN
@@
 $EndComp
 $Comp
-L GND-RESCUE-EtherDue #PWR518
+L GND-RESCUE-EtherDue #PWR073
 U 1 1 51663ACA
 P 6100 7250
-F 0 "#PWR518" H 6100 7250 30  0001 C CNN
+F 0 "#PWR073" H 6100 7250 30  0001 C CNN
 F 1 "GND" H 6100 7180 30  0001 C CNN
 F 2 "" H 6100 7250 60  0001 C CNN
@@
 1V8D
 $Comp
-L GND-RESCUE-EtherDue #PWR511
+L GND-RESCUE-EtherDue #PWR074
 U 1 1 51663AAD
 P 4100 7250
-F 0 "#PWR511" H 4100 7250 30  0001 C CNN
+F 0 "#PWR074" H 4100 7250 30  0001 C CNN
 F 1 "GND" H 4100 7180 30  0001 C CNN
 F 2 "" H 4100 7250 60  0001 C CNN
@@
 $EndComp
 $Comp
-L GND-RESCUE-EtherDue #PWR508
+L GND-RESCUE-EtherDue #PWR075
 U 1 1 51663A9A
 P 2900 7250
-F 0 "#PWR508" H 2900 7250 30  0001 C CNN
+F 0 "#PWR075" H 2900 7250 30  0001 C CNN
 F 1 "GND" H 2900 7180 30  0001 C CNN
 F 2 "" H 2900 7250 60  0001 C CNN
@@
 P 3500 6600
 F 0 "L601" H 3500 6550 40  0000 C CNN
-F 1 "1uH 250mA" H 3500 6700 40  0000 C CNN
+F 1 "WE-CBF-742792093" H 3500 6700 40  0000 C CNN
 F 2 "FT:0805" H 3500 6600 60  0001 C CNN
 F 3 "" H 3500 6600 60  0001 C CNN
@@
 P 4100 7000
 F 0 "C606" H 4150 7100 50  0000 L CNN
-F 1 "10uF 6.3V A TANT" V 3950 6650 50  0000 L CNN
+F 1 "10u/25V/X7R" V 3950 6650 50  0000 L CNN
 F 2 "SMD_Packages:SMD-1206_Pol" H 4100 7000 60  0001 C CNN
 F 3 "" H 4100 7000 60  0001 C CNN
@@
 P 2900 7000
 F 0 "C604" H 2950 7100 50  0000 L CNN
-F 1 "10uF 6.3V A TANT" V 2750 6650 50  0000 L CNN
+F 1 "10u/25V/X7R" V 2750 6650 50  0000 L CNN
 F 2 "SMD_Packages:SMD-1206_Pol" H 2900 7000 60  0001 C CNN
 F 3 "" H 2900 7000 60  0001 C CNN
@@
 Analog Power Decoupling\n
 $Comp
-L GND-RESCUE-EtherDue #PWR520
+L GND-RESCUE-EtherDue #PWR076
 U 1 1 516639AE
 P 6800 5200
-F 0 "#PWR520" H 6800 5200 30  0001 C CNN
+F 0 "#PWR076" H 6800 5200 30  0001 C CNN
 F 1 "GND" H 6800 5130 30  0001 C CNN
 F 2 "" H 6800 5200 60  0001 C CNN
@@
 $EndComp
 $Comp
-L +3.3V #PWR522
+L +3.3V #PWR077
 U 1 1 51663851
 P 7600 4200
-F 0 "#PWR522" H 7600 4160 30  0001 C CNN
+F 0 "#PWR077" H 7600 4160 30  0001 C CNN
 F 1 "+3.3V" H 7600 4310 30  0000 C CNN
 F 2 "" H 7600 4200 60  0001 C CNN
@@
 For DC PoE with low voltage,\njumper 3(PoE_V+) to 4(VIN)\n& 2(PoE_V-) to 1(GND)
 $Comp
-L GND-RESCUE-EtherDue #PWR505
+L GND-RESCUE-EtherDue #PWR078
 U 1 1 516634EC
 P 2100 7200
-F 0 "#PWR505" H 2100 7200 30  0001 C CNN
+F 0 "#PWR078" H 2100 7200 30  0001 C CNN
 F 1 "GND" H 2100 7130 30  0001 C CNN
 F 2 "" H 2100 7200 60  0001 C CNN
@@
 PoE Module Header
 $Comp
-L GND-RESCUE-EtherDue #PWR524
+L GND-RESCUE-EtherDue #PWR079
 U 1 1 51663438
 P 7600 5200
-F 0 "#PWR524" H 7600 5200 30  0001 C CNN
+F 0 "#PWR079" H 7600 5200 30  0001 C CNN
 F 1 "GND" H 7600 5130 30  0001 C CNN
 F 2 "" H 7600 5200 60  0001 C CNN
@@
 LINKLED
 $Comp
-L +3.3V #PWR523
+L +3.3V #PWR080
 U 1 1 51663302
 P 7600 4500
-F 0 "#PWR523" H 7600 4460 30  0001 C CNN
+F 0 "#PWR080" H 7600 4460 30  0001 C CNN
 F 1 "+3.3V" H 7600 4610 30  0000 C CNN
 F 2 "" H 7600 4500 60  0001 C CNN
@@
 $EndComp
 $Comp
-L GND-RESCUE-EtherDue #PWR521
+L GND-RESCUE-EtherDue #PWR081
 U 1 1 516632C9
 P 7250 4250
-F 0 "#PWR521" H 7250 4250 30  0001 C CNN
+F 0 "#PWR081" H 7250 4250 30  0001 C CNN
 F 1 "GND" H 7250 4180 30  0001 C CNN
 F 2 "" H 7250 4250 60  0001 C CNN
@@
 3V3A
 $Comp
-L GND-RESCUE-EtherDue #PWR507
+L GND-RESCUE-EtherDue #PWR082
 U 1 1 516630F1
 P 2750 1750
-F 0 "#PWR507" H 2750 1750 30  0001 C CNN
+F 0 "#PWR082" H 2750 1750 30  0001 C CNN
 F 1 "GND" H 2750 1680 30  0001 C CNN
 F 2 "" H 2750 1750 60  0001 C CNN
@@
 $EndComp
 $Comp
-L +3.3V #PWR509
+L +3.3V #PWR083
 U 1 1 516630E9
 P 3250 1050
-F 0 "#PWR509" H 3250 1010 30  0001 C CNN
+F 0 "#PWR083" H 3250 1010 30  0001 C CNN
 F 1 "+3.3V" H 3250 1160 30  0000 C CNN
 F 2 "" H 3250 1050 60  0001 C CNN
@@
 1.8v decoupling:\n1 near pins 15/16,\n1 near pin 33
 $Comp
-L GND-RESCUE-EtherDue #PWR510
+L GND-RESCUE-EtherDue #PWR084
 U 1 1 51662F42
 P 4050 1750
-F 0 "#PWR510" H 4050 1750 30  0001 C CNN
+F 0 "#PWR084" H 4050 1750 30  0001 C CNN
 F 1 "GND" H 4050 1680 30  0001 C CNN
 F 2 "" H 4050 1750 60  0001 C CNN
@@
 LINKLED
 $Comp
-L +3.3V #PWR525
+L +3.3V #PWR085
 U 1 1 51662070
 P 8050 750
-F 0 "#PWR525" H 8050 710 30  0001 C CNN
+F 0 "#PWR085" H 8050 710 30  0001 C CNN
 F 1 "+3.3V" H 8050 860 30  0000 C CNN
 F 2 "" H 8050 750 60  0001 C CNN
@@
 PWM2
 $Comp
-L GND-RESCUE-EtherDue #PWR502
+L GND-RESCUE-EtherDue #PWR086
 U 1 1 51661CDB
 P 1350 2950
-F 0 "#PWR502" H 1350 2950 30  0001 C CNN
+F 0 "#PWR086" H 1350 2950 30  0001 C CNN
 F 1 "GND" H 1350 2880 30  0001 C CNN
 F 2 "" H 1350 2950 60  0001 C CNN
@@
 WIZRST
 $Comp
-L GND-RESCUE-EtherDue #PWR513
+L GND-RESCUE-EtherDue #PWR087
 U 1 1 51661C24
 P 4400 1750
-F 0 "#PWR513" H 4400 1750 30  0001 C CNN
+F 0 "#PWR087" H 4400 1750 30  0001 C CNN
 F 1 "GND" H 4400 1680 30  0001 C CNN
 F 2 "" H 4400 1750 60  0001 C CNN
@@
 $EndComp
 $Comp
-L GND-RESCUE-EtherDue #PWR516
+L GND-RESCUE-EtherDue #PWR088
 U 1 1 51661C10
 P 5350 1950
-F 0 "#PWR516" H 5350 1950 30  0001 C CNN
+F 0 "#PWR088" H 5350 1950 30  0001 C CNN
 F 1 "GND" H 5350 1880 30  0001 C CNN
 F 2 "" H 5350 1950 60  0001 C CNN
@@
 $EndComp
 $Comp
-L GND-RESCUE-EtherDue #PWR519
+L GND-RESCUE-EtherDue #PWR089
 U 1 1 51661BE8
 P 6450 3900
-F 0 "#PWR519" H 6450 3900 30  0001 C CNN
+F 0 "#PWR089" H 6450 3900 30  0001 C CNN
 F 1 "GND" H 6450 3830 30  0001 C CNN
 F 2 "" H 6450 3900 60  0001 C CNN
@@
 $EndComp
 $Comp
-L GND-RESCUE-EtherDue #PWR517
+L GND-RESCUE-EtherDue #PWR090
 U 1 1 51661BC5
 P 5850 3900
-F 0 "#PWR517" H 5850 3900 30  0001 C CNN
+F 0 "#PWR090" H 5850 3900 30  0001 C CNN
 F 1 "GND" H 5850 3830 30  0001 C CNN
 F 2 "" H 5850 3900 60  0001 C CNN
@@
 $EndComp
 $Comp
-L GND-RESCUE-EtherDue #PWR512
+L GND-RESCUE-EtherDue #PWR091
 U 1 1 51661B99
 P 4300 5200
-F 0 "#PWR512" H 4300 5200 30  0001 C CNN
+F 0 "#PWR091" H 4300 5200 30  0001 C CNN
 F 1 "GND" H 4300 5130 30  0001 C CNN
 F 2 "" H 4300 5200 60  0001 C CNN
@@
 $EndComp
 $Comp
-L GND-RESCUE-EtherDue #PWR515
+L GND-RESCUE-EtherDue #PWR092
 U 1 1 51661B97
 P 5150 5650
-F 0 "#PWR515" H 5150 5650 30  0001 C CNN
+F 0 "#PWR092" H 5150 5650 30  0001 C CNN
 F 1 "GND" H 5150 5580 30  0001 C CNN
 F 2 "" H 5150 5650 60  0001 C CNN
@@
 $EndComp
 $Comp
-L GND-RESCUE-EtherDue #PWR506
+L GND-RESCUE-EtherDue #PWR093
 U 1 1 51661B24
 P 2350 4850
-F 0 "#PWR506" H 2350 4850 30  0001 C CNN
+F 0 "#PWR093" H 2350 4850 30  0001 C CNN
 F 1 "GND" H 2350 4780 30  0001 C CNN
 F 2 "" H 2350 4850 60  0001 C CNN
@@
 $EndComp
 $Comp
-L +3.3V #PWR501
+L +3.3V #PWR094
 U 1 1 51661B00
 P 1300 5850
-F 0 "#PWR501" H 1300 5810 30  0001 C CNN
+F 0 "#PWR094" H 1300 5810 30  0001 C CNN
 F 1 "+3.3V" H 1300 5960 30  0000 C CNN
 F 2 "" H 1300 5850 60  0001 C CNN
@@
 $EndComp
 $Comp
-L +3.3V #PWR503
+L +3.3V #PWR095
 U 1 1 5166191F
 P 1450 3700
-F 0 "#PWR503" H 1450 3660 30  0001 C CNN
+F 0 "#PWR095" H 1450 3660 30  0001 C CNN
 F 1 "+3.3V" H 1450 3810 30  0000 C CNN
 F 2 "" H 1450 3700 60  0001 C CNN
@@
 $EndComp
 $Comp
-L GND-RESCUE-EtherDue #PWR504
+L GND-RESCUE-EtherDue #PWR096
 U 1 1 516618BF
 P 1650 5000
-F 0 "#PWR504" H 1650 5000 30  0001 C CNN
+F 0 "#PWR096" H 1650 5000 30  0001 C CNN
 F 1 "GND" H 1650 4930 30  0001 C CNN
 F 2 "" H 1650 5000 60  0001 C CNN
