File: EtherDue_Power.sch (KiCad schematic (older format))
At the start: 48 parts, among them Q501 BC847BSMD, U203 LMV358IPWR, U501 POWERJACK, U502 LM2734Y, U503 FDN340P, U504 FDN340P, U505 NCP1117ST33T3G

Commit message: Rev B. Layout - Gerber/BOM need to be reexported
Parts:
- C501: footprint Capacitors_SMD:c_elec_5x5.3 -> Capacitors_SMD:c_elec_6.3x5.8
Changed lines of the file:
@@
 LIBS:w_transistor
 LIBS:w_logic
+LIBS:w_memory
 EELAYER 25 0
 EELAYER END
@@
 $EndDescr
 $Comp
-L PWR_FLAG #FLG701
+L PWR_FLAG #FLG0103
 U 1 1 5163B5CA
 P 1400 1400
-F 0 "#FLG701" H 1400 1495 30  0001 C CNN
+F 0 "#FLG0103" H 1400 1495 30  0001 C CNN
 F 1 "PWR_FLAG" H 1400 1580 30  0000 C CNN
 F 2 "" H 1400 1400 60  0001 C CNN
@@
 $EndComp
 $Comp
-L PWR_FLAG #FLG707
+L PWR_FLAG #FLG0104
 U 1 1 5163B2F3
 P 10450 4450
-F 0 "#FLG707" H 10450 4545 30  0001 C CNN
+F 0 "#FLG0104" H 10450 4545 30  0001 C CNN
 F 1 "PWR_FLAG" H 10450 4630 30  0000 C CNN
 F 2 "" H 10450 4450 60  0001 C CNN
@@
 $EndComp
 $Comp
-L PWR_FLAG #FLG706
+L PWR_FLAG #FLG0105
 U 1 1 5163B2EF
 P 10450 3800
-F 0 "#FLG706" H 10450 3895 30  0001 C CNN
+F 0 "#FLG0105" H 10450 3895 30  0001 C CNN
 F 1 "PWR_FLAG" H 10450 3980 30  0000 C CNN
 F 2 "" H 10450 3800 60  0001 C CNN
@@
 $EndComp
 $Comp
-L PWR_FLAG #FLG705
+L PWR_FLAG #FLG0106
 U 1 1 5163B2EB
 P 10450 2950
-F 0 "#FLG705" H 10450 3045 30  0001 C CNN
+F 0 "#FLG0106" H 10450 3045 30  0001 C CNN
 F 1 "PWR_FLAG" H 10450 3130 30  0000 C CNN
 F 2 "" H 10450 2950 60  0001 C CNN
@@
 VDDOUT
 $Comp
-L GND-RESCUE-EtherDue #PWR721
+L GND-RESCUE-EtherDue #PWR0107
 U 1 1 515CFFC7
 P 7800 6450
-F 0 "#PWR721" H 7800 6450 30  0001 C CNN
+F 0 "#PWR0107" H 7800 6450 30  0001 C CNN
 F 1 "GND" H 7800 6380 30  0001 C CNN
 F 2 "" H 7800 6450 60  0001 C CNN
@@
 $EndComp
 $Comp
-L GND-RESCUE-EtherDue #PWR720
+L GND-RESCUE-EtherDue #PWR0108
 U 1 1 515CFE6A
 P 7550 5800
-F 0 "#PWR720" H 7550 5800 30  0001 C CNN
+F 0 "#PWR0108" H 7550 5800 30  0001 C CNN
 F 1 "GND" H 7550 5730 30  0001 C CNN
 F 2 "" H 7550 5800 60  0001 C CNN
@@
 $EndComp
 $Comp
-L +3.3V #PWR719
+L +3.3V #PWR0109
 U 1 1 515CFE65
 P 7550 5250
-F 0 "#PWR719" H 7550 5210 30  0001 C CNN
+F 0 "#PWR0109" H 7550 5210 30  0001 C CNN
 F 1 "+3.3V" H 7550 5360 30  0000 C CNN
 F 2 "" H 7550 5250 60  0001 C CNN
@@
 $EndComp
 $Comp
-L +3.3V #PWR715
+L +3.3V #PWR0110
 U 1 1 515CFE50
 P 7450 3750
-F 0 "#PWR715" H 7450 3710 30  0001 C CNN
+F 0 "#PWR0110" H 7450 3710 30  0001 C CNN
 F 1 "+3.3V" H 7450 3860 30  0000 C CNN
 F 2 "" H 7450 3750 60  0001 C CNN
@@
 VDDOUTMI
 $Comp
-L GND-RESCUE-EtherDue #PWR718
+L GND-RESCUE-EtherDue #PWR0111
 U 1 1 515CFE4C
 P 7550 5050
-F 0 "#PWR718" H 7550 5050 30  0001 C CNN
+F 0 "#PWR0111" H 7550 5050 30  0001 C CNN
 F 1 "GND" H 7550 4980 30  0001 C CNN
 F 2 "" H 7550 5050 60  0001 C CNN
@@
 $EndComp
 $Comp
-L GND-RESCUE-EtherDue #PWR714
+L GND-RESCUE-EtherDue #PWR0112
 U 1 1 515CFDF7
 P 7450 3450
-F 0 "#PWR714" H 7450 3450 30  0001 C CNN
+F 0 "#PWR0112" H 7450 3450 30  0001 C CNN
 F 1 "GND" H 7450 3380 30  0001 C CNN
 F 2 "" H 7450 3450 60  0001 C CNN
@@
 $EndComp
 $Comp
-L +3.3V #PWR713
+L +3.3V #PWR0113
 U 1 1 515CFD93
 P 7450 2900
-F 0 "#PWR713" H 7450 2860 30  0001 C CNN
+F 0 "#PWR0113" H 7450 2860 30  0001 C CNN
 F 1 "+3.3V" H 7450 3010 30  0000 C CNN
 F 2 "" H 7450 2900 60  0001 C CNN
@@
 Forces off the power supply to USB port\nwhen the USB port is in HOST mode\n(and the board is powered from an external supply via VIN)
 $Comp
-L +5V #PWR708
+L +5V #PWR0114
 U 1 1 515CDDC3
 P 5200 4250
-F 0 "#PWR708" H 5200 4340 20  0001 C CNN
+F 0 "#PWR0114" H 5200 4340 20  0001 C CNN
 F 1 "+5V" H 5200 4340 30  0000 C CNN
 F 2 "" H 5200 4250 60  0001 C CNN
@@
 $EndComp
 $Comp
-L GND-RESCUE-EtherDue #PWR709
+L GND-RESCUE-EtherDue #PWR0115
 U 1 1 515CDD8D
 P 5200 5450
-F 0 "#PWR709" H 5200 5450 30  0001 C CNN
+F 0 "#PWR0115" H 5200 5450 30  0001 C CNN
 F 1 "GND" H 5200 5380 30  0001 C CNN
 F 2 "" H 5200 5450 60  0001 C CNN
@@
 +5V
 $Comp
-L GND-RESCUE-EtherDue #PWR710
+L GND-RESCUE-EtherDue #PWR0116
 U 1 1 515CDC85
 P 6150 7450
-F 0 "#PWR710" H 6150 7450 30  0001 C CNN
+F 0 "#PWR0116" H 6150 7450 30  0001 C CNN
 F 1 "GND" H 6150 7380 30  0001 C CNN
 F 2 "" H 6150 7450 60  0001 C CNN
@@
 CMP
 $Comp
-L +3.3V #PWR705
+L +3.3V #PWR0117
 U 1 1 515CDAC2
 P 4250 4300
-F 0 "#PWR705" H 4250 4260 30  0001 C CNN
+F 0 "#PWR0117" H 4250 4260 30  0001 C CNN
 F 1 "+3.3V" H 4250 4410 30  0000 C CNN
 F 2 "" H 4250 4300 60  0001 C CNN
@@
 $EndComp
 $Comp
-L PWR_FLAG #FLG703
+L PWR_FLAG #FLG0118
 U 1 1 515CDA13
 P 2550 1400
-F 0 "#FLG703" H 2550 1495 30  0001 C CNN
+F 0 "#FLG0118" H 2550 1495 30  0001 C CNN
 F 1 "PWR_FLAG" H 2550 1580 30  0000 C CNN
 F 2 "" H 2550 1400 60  0001 C CNN
@@
 $EndComp
 $Comp
-L GND-RESCUE-EtherDue #PWR706
+L GND-RESCUE-EtherDue #PWR0119
 U 1 1 515CD951
 P 4600 6100
-F 0 "#PWR706" H 4600 6100 30  0001 C CNN
+F 0 "#PWR0119" H 4600 6100 30  0001 C CNN
 F 1 "GND" H 4600 6030 30  0001 C CNN
 F 2 "" H 4600 6100 60  0001 C CNN
@@
 $EndComp
 $Comp
-L GND-RESCUE-EtherDue #PWR702
+L GND-RESCUE-EtherDue #PWR0120
 U 1 1 515CD94D
 P 2550 6300
-F 0 "#PWR702" H 2550 6300 30  0001 C CNN
+F 0 "#PWR0120" H 2550 6300 30  0001 C CNN
 F 1 "GND" H 2550 6230 30  0001 C CNN
 F 2 "" H 2550 6300 60  0001 C CNN
@@
 USB Power
 $Comp
-L +3.3V #PWR724
+L +3.3V #PWR0121
 U 1 1 515CD803
 P 10900 1000
-F 0 "#PWR724" H 10900 960 30  0001 C CNN
+F 0 "#PWR0121" H 10900 960 30  0001 C CNN
 F 1 "+3.3V" H 10900 1110 30  0000 C CNN
 F 2 "" H 10900 1000 60  0001 C CNN
@@
 $EndComp
 $Comp
-L GND-RESCUE-EtherDue #PWR723
+L GND-RESCUE-EtherDue #PWR0122
 U 1 1 515CD7D2
 P 10100 2200
-F 0 "#PWR723" H 10100 2200 30  0001 C CNN
+F 0 "#PWR0122" H 10100 2200 30  0001 C CNN
 F 1 "GND" H 10100 2130 30  0001 C CNN
 F 2 "" H 10100 2200 60  0001 C CNN
@@
 3.3V Regulator
 $Comp
-L PWR_FLAG #FLG704
+L PWR_FLAG #FLG0123
 U 1 1 515CD53B
 P 7400 1250
-F 0 "#FLG704" H 7400 1345 30  0001 C CNN
+F 0 "#FLG0123" H 7400 1345 30  0001 C CNN
 F 1 "PWR_FLAG" H 7400 1430 30  0000 C CNN
 F 2 "" H 7400 1250 60  0001 C CNN
@@
 $EndComp
 $Comp
-L GND-RESCUE-EtherDue #PWR722
+L GND-RESCUE-EtherDue #PWR0124
 U 1 1 515CD3F7
 P 8000 2300
-F 0 "#PWR722" H 8000 2300 30  0001 C CNN
+F 0 "#PWR0124" H 8000 2300 30  0001 C CNN
 F 1 "GND" H 8000 2230 30  0001 C CNN
 F 2 "" H 8000 2300 60  0001 C CNN
@@
 $EndComp
 $Comp
-L +5V #PWR717
+L +5V #PWR0125
 U 1 1 515CCC2C
 P 7550 1050
-F 0 "#PWR717" H 7550 1140 20  0001 C CNN
+F 0 "#PWR0125" H 7550 1140 20  0001 C CNN
 F 1 "+5V" H 7550 1140 30  0000 C CNN
 F 2 "" H 7550 1050 60  0001 C CNN
@@
 $EndComp
 $Comp
-L GND-RESCUE-EtherDue #PWR712
+L GND-RESCUE-EtherDue #PWR0126
 U 1 1 515CCC28
 P 6650 2300
-F 0 "#PWR712" H 6650 2300 30  0001 C CNN
+F 0 "#PWR0126" H 6650 2300 30  0001 C CNN
 F 1 "GND" H 6650 2230 30  0001 C CNN
 F 2 "" H 6650 2300 60  0001 C CNN
@@
 $EndComp
 $Comp
-L GND-RESCUE-EtherDue #PWR707
+L GND-RESCUE-EtherDue #PWR0127
 U 1 1 515CCC1E
 P 5000 1950
-F 0 "#PWR707" H 5000 1950 30  0001 C CNN
+F 0 "#PWR0127" H 5000 1950 30  0001 C CNN
 F 1 "GND" H 5000 1880 30  0001 C CNN
 F 2 "" H 5000 1950 60  0001 C CNN
@@
 $EndComp
 $Comp
-L GND-RESCUE-EtherDue #PWR703
+L GND-RESCUE-EtherDue #PWR0128
 U 1 1 515CCC19
 P 3450 1950
-F 0 "#PWR703" H 3450 1950 30  0001 C CNN
+F 0 "#PWR0128" H 3450 1950 30  0001 C CNN
 F 1 "GND" H 3450 1880 30  0001 C CNN
 F 2 "" H 3450 1950 60  0001 C CNN
@@
 5V Regulator
 $Comp
-L GND-RESCUE-EtherDue #PWR701
+L GND-RESCUE-EtherDue #PWR0129
 U 1 1 515CCB6C
 P 1600 2000
-F 0 "#PWR701" H 1600 2000 30  0001 C CNN
+F 0 "#PWR0129" H 1600 2000 30  0001 C CNN
 F 1 "GND" H 1600 1930 30  0001 C CNN
 F 2 "" H 1600 2000 60  0001 C CNN
@@
 F 0 "C501" H 2500 1800 50  0000 L CNN
 F 1 "47uF 25V" H 2500 1600 50  0000 L CNN
-F 2 "Capacitors_SMD:c_elec_5x5.3" H 2450 1700 60  0001 C CNN
+F 2 "Capacitors_SMD:c_elec_6.3x5.8" H 2450 1700 60  0001 C CNN
 F 3 "" H 2450 1700 60  0001 C CNN
 	1    2450 1700
@@
 Vin
 $Comp
-L GND-RESCUE-EtherDue #PWR711
+L GND-RESCUE-EtherDue #PWR0130
 U 1 1 5166FA0F
 P 6250 3400
-F 0 "#PWR711" H 6250 3400 30  0001 C CNN
+F 0 "#PWR0130" H 6250 3400 30  0001 C CNN
 F 1 "GND" H 6250 3330 30  0001 C CNN
 F 2 "" H 6250 3400 60  0000 C CNN
@@
 POWER_JACK
 $Comp
-L PWR_FLAG #FLG702
+L PWR_FLAG #FLG0131
 U 1 1 51666680
 P 2150 1900
-F 0 "#FLG702" H 2150 1995 30  0001 C CNN
+F 0 "#FLG0131" H 2150 1995 30  0001 C CNN
 F 1 "PWR_FLAG" H 2150 2080 30  0000 C CNN
 F 2 "" H 2150 1900 60  0000 C CNN
@@
 7-12V Recommended,\n6-20V Possible.
 $Comp
-L GND-RESCUE-EtherDue #PWR716
+L GND-RESCUE-EtherDue #PWR0132
 U 1 1 542492D2
 P 7500 4300
-F 0 "#PWR716" H 7500 4300 30  0001 C CNN
+F 0 "#PWR0132" H 7500 4300 30  0001 C CNN
 F 1 "GND" H 7500 4230 30  0001 C CNN
 F 2 "" H 7500 4300 60  0000 C CNN
@@
 $EndComp
 $Comp
-L GND-RESCUE-EtherDue #PWR704
+L GND-RESCUE-EtherDue #PWR0133
 U 1 1 54FE8130
 P 3850 1950
-F 0 "#PWR704" H 3850 1950 30  0001 C CNN
+F 0 "#PWR0133" H 3850 1950 30  0001 C CNN
 F 1 "GND" H 3850 1880 30  0001 C CNN
 F 2 "" H 3850 1950 60  0001 C CNN
