File: analog-level-adoption.sch (KiCad schematic (older format))
At the start: 30 parts

Commit message: 20150728
Parts:
- R2012: value TBD -> 6k8
Changed lines of the file:
@@
 P 7800 5600
 F 0 "R2012" V 7880 5600 50  0000 C CNN
-F 1 "TBD" V 7807 5601 50  0000 C CNN
+F 1 "6k8" V 7807 5601 50  0000 C CNN
 F 2 "Resistors_SMD:R_0603" V 7730 5600 30  0001 C CNN
 F 3 "" H 7800 5600 30  0000 C CNN

Commit message: Rev B. Layout - Gerber/BOM need to be reexported
Parts:
- R2010, R2011: value 6k8 -> DNP
Changed lines of the file:
@@
 LIBS:w_transistor
 LIBS:w_logic
+LIBS:w_memory
 EELAYER 25 0
 EELAYER END
@@
 P 7800 2550
 F 0 "R2010" V 7880 2550 50  0000 C CNN
-F 1 "6k8" V 7807 2551 50  0000 C CNN
+F 1 "DNP" V 7807 2551 50  0000 C CNN
 F 2 "Resistors_SMD:R_0603" V 7730 2550 30  0001 C CNN
 F 3 "" H 7800 2550 30  0000 C CNN
@@
 $EndComp
 $Comp
-L GND-RESCUE-EtherDue #PWR2013
+L GND-RESCUE-EtherDue #PWR0377
 U 1 1 55326E08
 P 7800 2800
-F 0 "#PWR2013" H 7800 2550 60  0001 C CNN
+F 0 "#PWR0377" H 7800 2550 60  0001 C CNN
 F 1 "GND" H 7800 2650 60  0000 C CNN
 F 2 "" H 7800 2800 60  0000 C CNN
@@
 $EndComp
 $Comp
-L GND-RESCUE-EtherDue #PWR2016
+L GND-RESCUE-EtherDue #PWR0378
 U 1 1 55326E23
 P 8000 2800
-F 0 "#PWR2016" H 8000 2550 60  0001 C CNN
+F 0 "#PWR0378" H 8000 2550 60  0001 C CNN
 F 1 "GND" H 8000 2650 60  0000 C CNN
 F 2 "" H 8000 2800 60  0000 C CNN
@@
 P 7800 4100
 F 0 "R2011" V 7880 4100 50  0000 C CNN
-F 1 "6k8" V 7807 4101 50  0000 C CNN
+F 1 "DNP" V 7807 4101 50  0000 C CNN
 F 2 "Resistors_SMD:R_0603" V 7730 4100 30  0001 C CNN
 F 3 "" H 7800 4100 30  0000 C CNN
@@
 $EndComp
 $Comp
-L GND-RESCUE-EtherDue #PWR2014
+L GND-RESCUE-EtherDue #PWR0379
 U 1 1 5532725C
 P 7800 4350
-F 0 "#PWR2014" H 7800 4100 60  0001 C CNN
+F 0 "#PWR0379" H 7800 4100 60  0001 C CNN
 F 1 "GND" H 7800 4200 60  0000 C CNN
 F 2 "" H 7800 4350 60  0000 C CNN
@@
 $EndComp
 $Comp
-L GND-RESCUE-EtherDue #PWR2017
+L GND-RESCUE-EtherDue #PWR0380
 U 1 1 55327262
 P 8000 4350
-F 0 "#PWR2017" H 8000 4100 60  0001 C CNN
+F 0 "#PWR0380" H 8000 4100 60  0001 C CNN
 F 1 "GND" H 8000 4200 60  0000 C CNN
 F 2 "" H 8000 4350 60  0000 C CNN
@@
 $EndComp
 $Comp
-L GND-RESCUE-EtherDue #PWR2015
+L GND-RESCUE-EtherDue #PWR0381
 U 1 1 55327405
 P 7800 5850
-F 0 "#PWR2015" H 7800 5600 60  0001 C CNN
+F 0 "#PWR0381" H 7800 5600 60  0001 C CNN
 F 1 "GND" H 7800 5700 60  0000 C CNN
 F 2 "" H 7800 5850 60  0000 C CNN
@@
 $EndComp
 $Comp
-L GND-RESCUE-EtherDue #PWR2018
+L GND-RESCUE-EtherDue #PWR0382
 U 1 1 5532740B
 P 8000 5850
-F 0 "#PWR2018" H 8000 5600 60  0001 C CNN
+F 0 "#PWR0382" H 8000 5600 60  0001 C CNN
 F 1 "GND" H 8000 5700 60  0000 C CNN
 F 2 "" H 8000 5850 60  0000 C CNN
@@
 $EndComp
 $Comp
-L GND-RESCUE-EtherDue #PWR2001
+L GND-RESCUE-EtherDue #PWR0383
 U 1 1 5532829E
 P 3400 2800
-F 0 "#PWR2001" H 3400 2550 60  0001 C CNN
+F 0 "#PWR0383" H 3400 2550 60  0001 C CNN
 F 1 "GND" H 3400 2650 60  0000 C CNN
 F 2 "" H 3400 2800 60  0000 C CNN
@@
 $EndComp
 $Comp
-L GND-RESCUE-EtherDue #PWR2004
+L GND-RESCUE-EtherDue #PWR0384
 U 1 1 553282A4
 P 3600 2800
-F 0 "#PWR2004" H 3600 2550 60  0001 C CNN
+F 0 "#PWR0384" H 3600 2550 60  0001 C CNN
 F 1 "GND" H 3600 2650 60  0000 C CNN
 F 2 "" H 3600 2800 60  0000 C CNN
@@
 Connection ~ 4500 2200
 $Comp
-L GND-RESCUE-EtherDue #PWR2007
+L GND-RESCUE-EtherDue #PWR0385
 U 1 1 553287E6
 P 4300 2800
-F 0 "#PWR2007" H 4300 2550 60  0001 C CNN
+F 0 "#PWR0385" H 4300 2550 60  0001 C CNN
 F 1 "GND" H 4300 2650 60  0000 C CNN
 F 2 "" H 4300 2800 60  0000 C CNN
@@
 $EndComp
 $Comp
-L GND-RESCUE-EtherDue #PWR2002
+L GND-RESCUE-EtherDue #PWR0386
 U 1 1 55329BEC
 P 3400 4350
-F 0 "#PWR2002" H 3400 4100 60  0001 C CNN
+F 0 "#PWR0386" H 3400 4100 60  0001 C CNN
 F 1 "GND" H 3400 4200 60  0000 C CNN
 F 2 "" H 3400 4350 60  0000 C CNN
@@
 $EndComp
 $Comp
-L GND-RESCUE-EtherDue #PWR2005
+L GND-RESCUE-EtherDue #PWR0387
 U 1 1 55329BF2
 P 3600 4350
-F 0 "#PWR2005" H 3600 4100 60  0001 C CNN
+F 0 "#PWR0387" H 3600 4100 60  0001 C CNN
 F 1 "GND" H 3600 4200 60  0000 C CNN
 F 2 "" H 3600 4350 60  0000 C CNN
@@
 Connection ~ 4500 3750
 $Comp
-L GND-RESCUE-EtherDue #PWR2008
+L GND-RESCUE-EtherDue #PWR0388
 U 1 1 55329C08
 P 4300 4350
-F 0 "#PWR2008" H 4300 4100 60  0001 C CNN
+F 0 "#PWR0388" H 4300 4100 60  0001 C CNN
 F 1 "GND" H 4300 4200 60  0000 C CNN
 F 2 "" H 4300 4350 60  0000 C CNN
@@
 $EndComp
 $Comp
-L GND-RESCUE-EtherDue #PWR2003
+L GND-RESCUE-EtherDue #PWR0389
 U 1 1 55329E60
 P 3400 5850
-F 0 "#PWR2003" H 3400 5600 60  0001 C CNN
+F 0 "#PWR0389" H 3400 5600 60  0001 C CNN
 F 1 "GND" H 3400 5700 60  0000 C CNN
 F 2 "" H 3400 5850 60  0000 C CNN
@@
 $EndComp
 $Comp
-L GND-RESCUE-EtherDue #PWR2006
+L GND-RESCUE-EtherDue #PWR0390
 U 1 1 55329E66
 P 3600 5850
-F 0 "#PWR2006" H 3600 5600 60  0001 C CNN
+F 0 "#PWR0390" H 3600 5600 60  0001 C CNN
 F 1 "GND" H 3600 5700 60  0000 C CNN
 F 2 "" H 3600 5850 60  0000 C CNN
@@
 Connection ~ 4500 5250
 $Comp
-L GND-RESCUE-EtherDue #PWR2009
+L GND-RESCUE-EtherDue #PWR0391
 U 1 1 55329E7C
 P 4300 5850
-F 0 "#PWR2009" H 4300 5600 60  0001 C CNN
+F 0 "#PWR0391" H 4300 5600 60  0001 C CNN
 F 1 "GND" H 4300 5700 60  0000 C CNN
 F 2 "" H 4300 5850 60  0000 C CNN
@@
 $EndComp
 $Comp
-L GND-RESCUE-EtherDue #PWR2019
+L GND-RESCUE-EtherDue #PWR0392
 U 1 1 54F6FA20
 P 8600 5850
-F 0 "#PWR2019" H 8600 5600 60  0001 C CNN
+F 0 "#PWR0392" H 8600 5600 60  0001 C CNN
 F 1 "GND" H 8600 5700 60  0000 C CNN
 F 2 "" H 8600 5850 60  0000 C CNN
@@
 $EndComp
 $Comp
-L GND-RESCUE-EtherDue #PWR2010
+L GND-RESCUE-EtherDue #PWR0393
 U 1 1 54F8DCA3
 P 4650 2800
-F 0 "#PWR2010" H 4650 2550 60  0001 C CNN
+F 0 "#PWR0393" H 4650 2550 60  0001 C CNN
 F 1 "GND" H 4650 2650 60  0000 C CNN
 F 2 "" H 4650 2800 60  0000 C CNN
@@
 $EndComp
 $Comp
-L GND-RESCUE-EtherDue #PWR2011
+L GND-RESCUE-EtherDue #PWR0394
 U 1 1 54F8DE19
 P 4650 4350
-F 0 "#PWR2011" H 4650 4100 60  0001 C CNN
+F 0 "#PWR0394" H 4650 4100 60  0001 C CNN
 F 1 "GND" H 4650 4200 60  0000 C CNN
 F 2 "" H 4650 4350 60  0000 C CNN
@@
 $EndComp
 $Comp
-L GND-RESCUE-EtherDue #PWR2012
+L GND-RESCUE-EtherDue #PWR0395
 U 1 1 54F8DFAA
 P 4650 5850
-F 0 "#PWR2012" H 4650 5600 60  0001 C CNN
+F 0 "#PWR0395" H 4650 5600 60  0001 C CNN
 F 1 "GND" H 4650 5700 60  0000 C CNN
 F 2 "" H 4650 5850 60  0000 C CNN
@@
 $EndComp
 $Comp
-L GND-RESCUE-EtherDue #PWR2020
+L GND-RESCUE-EtherDue #PWR0396
 U 1 1 54F8E6EA
 P 8950 5850
-F 0 "#PWR2020" H 8950 5600 60  0001 C CNN
+F 0 "#PWR0396" H 8950 5600 60  0001 C CNN
 F 1 "GND" H 8950 5700 60  0000 C CNN
 F 2 "" H 8950 5850 60  0000 C CNN
