File: can-bus.sch (KiCad schematic (older format))
At the start: 15 parts, among them P901 677006144621, P902 677006144621, U901 TJA1040T

Commit message: Rev B. Layout - Gerber/BOM need to be reexported
Parts:
- R904, R905: footprint Resistors_SMD:R_1206 -> Resistors_SMD:R_0805
- R906, R907: footprint Resistors_SMD:R_0603 -> Resistors_SMD:R_0805
Changed lines of the file:
@@
 LIBS:w_transistor
 LIBS:w_logic
+LIBS:w_memory
 EELAYER 25 0
 EELAYER END
@@
 	4200 4150 4200 4200
 $Comp
-L GND-RESCUE-EtherDue #PWR903
+L GND-RESCUE-EtherDue #PWR0158
 U 1 1 54F00676
 P 4200 4800
-F 0 "#PWR903" H 4200 4550 60  0001 C CNN
+F 0 "#PWR0158" H 4200 4550 60  0001 C CNN
 F 1 "GND" H 4200 4650 60  0000 C CNN
 F 2 "" H 4200 4800 60  0000 C CNN
@@
 	4200 4800 4200 4700
 $Comp
-L GND-RESCUE-EtherDue #PWR904
+L GND-RESCUE-EtherDue #PWR0159
 U 1 1 54F006A8
 P 4800 4800
-F 0 "#PWR904" H 4800 4550 60  0001 C CNN
+F 0 "#PWR0159" H 4800 4550 60  0001 C CNN
 F 1 "GND" H 4800 4650 60  0000 C CNN
 F 2 "" H 4800 4800 60  0000 C CNN
@@
 $EndComp
 $Comp
-L GND-RESCUE-EtherDue #PWR902
+L GND-RESCUE-EtherDue #PWR0160
 U 1 1 54F007D4
 P 3550 4800
-F 0 "#PWR902" H 3550 4550 60  0001 C CNN
+F 0 "#PWR0160" H 3550 4550 60  0001 C CNN
 F 1 "GND" H 3550 4650 60  0000 C CNN
 F 2 "" H 3550 4800 60  0000 C CNN
@@
 F 0 "R904" V 6180 3750 50  0000 C CNN
 F 1 "60R" V 6107 3751 50  0000 C CNN
-F 2 "Resistors_SMD:R_1206" V 6030 3750 30  0000 C CNN
+F 2 "Resistors_SMD:R_0805" V 6030 3750 30  0000 C CNN
 F 3 "" H 6100 3750 30  0000 C CNN
 	1    6100 3750
@@
 F 0 "R905" V 6180 4250 50  0000 C CNN
 F 1 "60R" V 6107 4251 50  0000 C CNN
-F 2 "Resistors_SMD:R_1206" V 6030 4250 30  0000 C CNN
+F 2 "Resistors_SMD:R_0805" V 6030 4250 30  0000 C CNN
 F 3 "" H 6100 4250 30  0000 C CNN
 	1    6100 4250
@@
 F 0 "R906" V 6780 3750 50  0000 C CNN
 F 1 "1k3" V 6707 3751 50  0000 C CNN
-F 2 "Resistors_SMD:R_0603" V 6630 3750 30  0001 C CNN
+F 2 "Resistors_SMD:R_0805" V 6630 3750 30  0001 C CNN
 F 3 "" H 6700 3750 30  0000 C CNN
 	1    6700 3750
@@
 F 0 "R907" V 6780 4250 50  0000 C CNN
 F 1 "1k3" V 6707 4251 50  0000 C CNN
-F 2 "Resistors_SMD:R_0603" V 6630 4250 30  0001 C CNN
+F 2 "Resistors_SMD:R_0805" V 6630 4250 30  0001 C CNN
 F 3 "" H 6700 4250 30  0000 C CNN
 	1    6700 4250
@@
 	10050 4350 9200 4350
 $Comp
-L GND-RESCUE-EtherDue #PWR907
+L GND-RESCUE-EtherDue #PWR0161
 U 1 1 54F016F8
 P 9200 4350
-F 0 "#PWR907" H 9200 4100 60  0001 C CNN
+F 0 "#PWR0161" H 9200 4100 60  0001 C CNN
 F 1 "GND" H 9200 4200 60  0000 C CNN
 F 2 "" H 9200 4350 60  0000 C CNN
@@
 $EndComp
 $Comp
-L GND-RESCUE-EtherDue #PWR906
+L GND-RESCUE-EtherDue #PWR0162
 U 1 1 54F01715
 P 9150 3300
-F 0 "#PWR906" H 9150 3050 60  0001 C CNN
+F 0 "#PWR0162" H 9150 3050 60  0001 C CNN
 F 1 "GND" H 9150 3150 60  0000 C CNN
 F 2 "" H 9150 3300 60  0000 C CNN
@@
 Firewire Connectors\nare used for CAN
 $Comp
-L GND-RESCUE-EtherDue #PWR905
+L GND-RESCUE-EtherDue #PWR0163
 U 1 1 54F01A23
 P 7600 4000
-F 0 "#PWR905" H 7600 3750 60  0001 C CNN
+F 0 "#PWR0163" H 7600 3750 60  0001 C CNN
 F 1 "GND" H 7600 3850 60  0000 C CNN
 F 2 "" H 7600 4000 60  0000 C CNN
@@
 	2600 4050 2600 4200
 $Comp
-L GND-RESCUE-EtherDue #PWR901
+L GND-RESCUE-EtherDue #PWR0164
 U 1 1 54F021C9
 P 2600 4800
-F 0 "#PWR901" H 2600 4550 60  0001 C CNN
+F 0 "#PWR0164" H 2600 4550 60  0001 C CNN
 F 1 "GND" H 2600 4650 60  0000 C CNN
 F 2 "" H 2600 4800 60  0000 C CNN
@@
 	8800 4450 8800 4150
 $Comp
-L GND-RESCUE-EtherDue #PWR909
+L GND-RESCUE-EtherDue #PWR0165
 U 1 1 55548402
 P 9750 5200
-F 0 "#PWR909" H 9750 4950 60  0001 C CNN
+F 0 "#PWR0165" H 9750 4950 60  0001 C CNN
 F 1 "GND" H 9750 5050 60  0000 C CNN
 F 2 "" H 9750 5200 60  0000 C CNN
@@
 Connection ~ 9750 4950
 $Comp
-L GND-RESCUE-EtherDue #PWR908
+L GND-RESCUE-EtherDue #PWR0166
 U 1 1 555485A9
 P 9750 4150
-F 0 "#PWR908" H 9750 3900 60  0001 C CNN
+F 0 "#PWR0166" H 9750 3900 60  0001 C CNN
 F 1 "GND" H 9750 4000 60  0000 C CNN
 F 2 "" H 9750 4150 60  0000 C CNN
