File: pa-monitor-power.sch (KiCad schematic (older format))
At the start: 48 parts, among them P801 MSTBV2, U801 TPS7A4501DCQT, U802 TPS7A4501DCQT, U803 TPS7A4501DCQT, U804 REG101NA-5

Commit message: 20150728
Parts:
- L802, L803: value WE-CBF-742792093 -> WE-CBF-742792040
Changed lines of the file:
@@
 P 3000 750
 F 0 "L802" H 3000 850 50  0000 C CNN
-F 1 "WE-CBF-742792093" H 3000 700 50  0000 C CNN
+F 1 "WE-CBF-742792040" H 3000 700 50  0000 C CNN
 F 2 "Resistors_SMD:R_0805" H 2850 600 40  0000 C CNN
 F 3 "" H 3000 750 60  0000 C CNN
@@
 P 3000 1150
 F 0 "L803" H 3000 1250 50  0000 C CNN
-F 1 "WE-CBF-742792093" H 3000 1100 50  0000 C CNN
+F 1 "WE-CBF-742792040" H 3000 1100 50  0000 C CNN
 F 2 "Resistors_SMD:R_0805" H 2850 1000 40  0000 C CNN
 F 3 "" H 3000 1150 60  0000 C CNN

Commit message: Rev B. Layout - Gerber/BOM need to be reexported
Parts:
- F801: value SMD100F -> SMD050F; footprint eagle-switch-raychem:SMD050F -> zeilhofer:SMD050F
Changed lines of the file:
@@
 LIBS:w_transistor
 LIBS:w_logic
+LIBS:w_memory
 EELAYER 25 0
 EELAYER END
@@
 $EndComp
 $Comp
-L GND-RESCUE-EtherDue #PWR802
+L GND-RESCUE-EtherDue #PWR0134
 U 1 1 54EDC972
 P 1600 2700
-F 0 "#PWR802" H 1600 2450 60  0001 C CNN
+F 0 "#PWR0134" H 1600 2450 60  0001 C CNN
 F 1 "GND" H 1600 2550 60  0000 C CNN
 F 2 "" H 1600 2700 60  0000 C CNN
@@
 P 1900 2100
 F 0 "F801" H 1800 2250 40  0000 C CNN
-F 1 "SMD100F" H 1900 1950 40  0000 C CNN
-F 2 "eagle-switch-raychem:SMD050F" H 1900 2100 60  0001 C CNN
+F 1 "SMD050F" H 1900 1950 40  0000 C CNN
+F 2 "zeilhofer:SMD050F" H 1900 2100 60  0001 C CNN
 F 3 "" H 1900 2100 60  0000 C CNN
 	1    1900 2100
@@
 $EndComp
 $Comp
-L PWR_FLAG #FLG801
+L PWR_FLAG #FLG0135
 U 1 1 54EDE151
 P 3450 2000
-F 0 "#FLG801" H 3450 2095 30  0001 C CNN
+F 0 "#FLG0135" H 3450 2095 30  0001 C CNN
 F 1 "PWR_FLAG" H 3450 2180 30  0000 C CNN
 F 2 "" H 3450 2000 60  0000 C CNN
@@
 $EndComp
 $Comp
-L GND-RESCUE-EtherDue #PWR809
+L GND-RESCUE-EtherDue #PWR0136
 U 1 1 54EED3C1
 P 7200 2450
-F 0 "#PWR809" H 7200 2200 60  0001 C CNN
+F 0 "#PWR0136" H 7200 2200 60  0001 C CNN
 F 1 "GND" H 7200 2300 60  0000 C CNN
 F 2 "" H 7200 2450 60  0000 C CNN
@@
 $EndComp
 $Comp
-L GND-RESCUE-EtherDue #PWR816
+L GND-RESCUE-EtherDue #PWR0137
 U 1 1 54EED683
 P 9200 2450
-F 0 "#PWR816" H 9200 2200 60  0001 C CNN
+F 0 "#PWR0137" H 9200 2200 60  0001 C CNN
 F 1 "GND" H 9200 2300 60  0000 C CNN
 F 2 "" H 9200 2450 60  0000 C CNN
@@
 1.21V
 $Comp
-L GND-RESCUE-EtherDue #PWR805
+L GND-RESCUE-EtherDue #PWR0138
 U 1 1 54EEDE58
 P 6150 2450
-F 0 "#PWR805" H 6150 2200 60  0001 C CNN
+F 0 "#PWR0138" H 6150 2200 60  0001 C CNN
 F 1 "GND" H 6150 2300 60  0000 C CNN
 F 2 "" H 6150 2450 60  0000 C CNN
@@
 $EndComp
 $Comp
-L GND-RESCUE-EtherDue #PWR810
+L GND-RESCUE-EtherDue #PWR0139
 U 1 1 54EEEA64
 P 7200 3650
-F 0 "#PWR810" H 7200 3400 60  0001 C CNN
+F 0 "#PWR0139" H 7200 3400 60  0001 C CNN
 F 1 "GND" H 7200 3500 60  0000 C CNN
 F 2 "" H 7200 3650 60  0000 C CNN
@@
 $EndComp
 $Comp
-L GND-RESCUE-EtherDue #PWR817
+L GND-RESCUE-EtherDue #PWR0140
 U 1 1 54EEEA7D
 P 9200 3650
-F 0 "#PWR817" H 9200 3400 60  0001 C CNN
+F 0 "#PWR0140" H 9200 3400 60  0001 C CNN
 F 1 "GND" H 9200 3500 60  0000 C CNN
 F 2 "" H 9200 3650 60  0000 C CNN
@@
 1.21V
 $Comp
-L GND-RESCUE-EtherDue #PWR806
+L GND-RESCUE-EtherDue #PWR0141
 U 1 1 54EEEA8F
 P 6150 3650
-F 0 "#PWR806" H 6150 3400 60  0001 C CNN
+F 0 "#PWR0141" H 6150 3400 60  0001 C CNN
 F 1 "GND" H 6150 3500 60  0000 C CNN
 F 2 "" H 6150 3650 60  0000 C CNN
@@
 $EndComp
 $Comp
-L GND-RESCUE-EtherDue #PWR811
+L GND-RESCUE-EtherDue #PWR0142
 U 1 1 54EEEC2A
 P 7200 4850
-F 0 "#PWR811" H 7200 4600 60  0001 C CNN
+F 0 "#PWR0142" H 7200 4600 60  0001 C CNN
 F 1 "GND" H 7200 4700 60  0000 C CNN
 F 2 "" H 7200 4850 60  0000 C CNN
@@
 $EndComp
 $Comp
-L GND-RESCUE-EtherDue #PWR818
+L GND-RESCUE-EtherDue #PWR0143
 U 1 1 54EEEC43
 P 9200 4850
-F 0 "#PWR818" H 9200 4600 60  0001 C CNN
+F 0 "#PWR0143" H 9200 4600 60  0001 C CNN
 F 1 "GND" H 9200 4700 60  0000 C CNN
 F 2 "" H 9200 4850 60  0000 C CNN
@@
 1.21V
 $Comp
-L GND-RESCUE-EtherDue #PWR807
+L GND-RESCUE-EtherDue #PWR0144
 U 1 1 54EEEC55
 P 6150 4850
-F 0 "#PWR807" H 6150 4600 60  0001 C CNN
+F 0 "#PWR0144" H 6150 4600 60  0001 C CNN
 F 1 "GND" H 6150 4700 60  0000 C CNN
 F 2 "" H 6150 4850 60  0000 C CNN
@@
 $EndComp
 $Comp
-L GND-RESCUE-EtherDue #PWR808
+L GND-RESCUE-EtherDue #PWR0145
 U 1 1 54EF9E9A
 P 6150 6200
-F 0 "#PWR808" H 6150 5950 60  0001 C CNN
+F 0 "#PWR0145" H 6150 5950 60  0001 C CNN
 F 1 "GND" H 6150 6050 60  0000 C CNN
 F 2 "" H 6150 6200 60  0000 C CNN
@@
 $EndComp
 $Comp
-L GND-RESCUE-EtherDue #PWR812
+L GND-RESCUE-EtherDue #PWR0146
 U 1 1 54EF9EC5
 P 7200 6200
-F 0 "#PWR812" H 7200 5950 60  0001 C CNN
+F 0 "#PWR0146" H 7200 5950 60  0001 C CNN
 F 1 "GND" H 7200 6050 60  0000 C CNN
 F 2 "" H 7200 6200 60  0000 C CNN
@@
 $EndComp
 $Comp
-L GND-RESCUE-EtherDue #PWR813
+L GND-RESCUE-EtherDue #PWR0147
 U 1 1 54EF9EF0
 P 7750 6200
-F 0 "#PWR813" H 7750 5950 60  0001 C CNN
+F 0 "#PWR0147" H 7750 5950 60  0001 C CNN
 F 1 "GND" H 7750 6050 60  0000 C CNN
 F 2 "" H 7750 6200 60  0000 C CNN
@@
 $EndComp
 $Comp
-L GND-RESCUE-EtherDue #PWR814
+L GND-RESCUE-EtherDue #PWR0148
 U 1 1 54EF9F1B
 P 8350 6200
-F 0 "#PWR814" H 8350 5950 60  0001 C CNN
+F 0 "#PWR0148" H 8350 5950 60  0001 C CNN
 F 1 "GND" H 8350 6050 60  0000 C CNN
 F 2 "" H 8350 6200 60  0000 C CNN
@@
 $EndComp
 $Comp
-L GND-RESCUE-EtherDue #PWR815
+L GND-RESCUE-EtherDue #PWR0149
 U 1 1 552030B4
 P 8850 6200
-F 0 "#PWR815" H 8850 5950 60  0001 C CNN
+F 0 "#PWR0149" H 8850 5950 60  0001 C CNN
 F 1 "GND" H 8850 6050 60  0000 C CNN
 F 2 "" H 8850 6200 60  0000 C CNN
@@
 $EndComp
 $Comp
-L GND-RESCUE-EtherDue #PWR803
+L GND-RESCUE-EtherDue #PWR0150
 U 1 1 54FBFF34
 P 4550 1900
-F 0 "#PWR803" H 4550 1650 60  0001 C CNN
+F 0 "#PWR0150" H 4550 1650 60  0001 C CNN
 F 1 "GND" H 4550 1750 60  0000 C CNN
 F 2 "" H 4550 1900 60  0000 C CNN
@@
 $EndComp
 $Comp
-L GND-RESCUE-EtherDue #PWR804
+L GND-RESCUE-EtherDue #PWR0151
 U 1 1 54FBFF69
 P 5000 1900
-F 0 "#PWR804" H 5000 1650 60  0001 C CNN
+F 0 "#PWR0151" H 5000 1650 60  0001 C CNN
 F 1 "GND" H 5000 1750 60  0000 C CNN
 F 2 "" H 5000 1900 60  0000 C CNN
@@
 $EndComp
 $Comp
-L PWR_FLAG #FLG804
+L PWR_FLAG #FLG0152
 U 1 1 550AA277
 P 10350 1800
-F 0 "#FLG804" H 10350 1895 30  0001 C CNN
+F 0 "#FLG0152" H 10350 1895 30  0001 C CNN
 F 1 "PWR_FLAG" H 10350 1980 30  0000 C CNN
 F 2 "" H 10350 1800 60  0000 C CNN
@@
 $EndComp
 $Comp
-L PWR_FLAG #FLG805
+L PWR_FLAG #FLG0153
 U 1 1 550AAAF5
 P 10350 3000
-F 0 "#FLG805" H 10350 3095 30  0001 C CNN
+F 0 "#FLG0153" H 10350 3095 30  0001 C CNN
 F 1 "PWR_FLAG" H 10350 3180 30  0000 C CNN
 F 2 "" H 10350 3000 60  0000 C CNN
@@
 $EndComp
 $Comp
-L PWR_FLAG #FLG806
+L PWR_FLAG #FLG0154
 U 1 1 550AAB05
 P 10350 4200
-F 0 "#FLG806" H 10350 4295 30  0001 C CNN
+F 0 "#FLG0154" H 10350 4295 30  0001 C CNN
 F 1 "PWR_FLAG" H 10350 4380 30  0000 C CNN
 F 2 "" H 10350 4200 60  0000 C CNN
@@
 $EndComp
 $Comp
-L PWR_FLAG #FLG802
+L PWR_FLAG #FLG0155
 U 1 1 550AE7D6
 P 10350 750
-F 0 "#FLG802" H 10350 845 30  0001 C CNN
+F 0 "#FLG0155" H 10350 845 30  0001 C CNN
 F 1 "PWR_FLAG" H 10350 930 30  0000 C CNN
 F 2 "" H 10350 750 60  0000 C CNN
@@
 $EndComp
 $Comp
-L PWR_FLAG #FLG803
+L PWR_FLAG #FLG0156
 U 1 1 550AE80D
 P 10350 1150
-F 0 "#FLG803" H 10350 1245 30  0001 C CNN
+F 0 "#FLG0156" H 10350 1245 30  0001 C CNN
 F 1 "PWR_FLAG" H 10350 1330 30  0000 C CNN
 F 2 "" H 10350 1150 60  0000 C CNN
@@
 $EndComp
 $Comp
-L GND-RESCUE-EtherDue #PWR801
+L GND-RESCUE-EtherDue #PWR0157
 U 1 1 5558B664
 P 1000 1750
-F 0 "#PWR801" H 1000 1500 60  0001 C CNN
+F 0 "#PWR0157" H 1000 1500 60  0001 C CNN
 F 1 "GND" H 1000 1600 60  0000 C CNN
 F 2 "" H 1000 1750 60  0000 C CNN
